File: pcb/Sigma1.kicad_pcb (KiCad board)
At the start: 2 copper layers, 48 x 78 mm, 60 parts, among them J1 Conn_01x02, J10 Screw_Terminal_01x02, J11 Screw_Terminal_01x02, J2 Screw_Terminal_01x02, J3 Servo 1, J4 Servo 2, J5 Servo 3, J6 Servo 1, J8 Conn_01x10, J9 Screw_Terminal_01x02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

Commit message: supply chain changes
Parts:
- removed SW2: SW_Push, Button_Switch_SMD:SW_SPST_B3U-1000P-B
- removed U4: MS5611-01BA, Package_LGA:LGA-8_3x5mm_P1.25mm
- added C6: 100n, Capacitor_SMD:C_0603_1608Metric, F.Cu at (27.6, 33.9)
- added SW3: TS-1088R-02026, easyeda2kicad:SW-SMD_L3.9-W3.0-P4.45, F.Cu at (20.9, 23.5)
- added U7: MLX90395KDC-BBA-001-SP, MLX90395KDC-BBA-001-SP:SOIC127P600X172-8N, F.Cu at (37.1, 34.6)
- C19: renamed from C6; value C -> 10uf
- C5: value C -> 0.1μF
- J3, J4, J5, J6: footprint Connector_PinHeader_2.54mm:PinHeader_1x03_P2.54mm_Vertical_SMD_Pin1Left -> Connector_PinHeader_2.54mm:PinHeader_1x03_P2.54mm_Vertical
- J8: footprint Connector_PinSocket_2.54mm:PinSocket_1x10_P2.54mm_Vertical_SMD_Pin1Left -> Connector_PinHeader_2.54mm:PinHeader_1x10_P2.54mm_Vertical
- R4: value 350 -> 330
- SW1: value SW_Push -> TS-1088R-02026; footprint Button_Switch_SMD:SW_SPST_B3U-1000P-B -> easyeda2kicad:SW-SMD_L3.9-W3.0-P4.45
- U5: value MLX90395xLW -> BMP390_C5124834; footprint Package_DFN_QFN:QFN-16-1EP_3x3mm_P0.5mm_EP1.675x1.675mm -> easyeda2kicad:LGA-10_L2.0-W2.0-P0.50-BL
- moved SW1 31.7 mm to (47.9, 34.7), turned to 180 degrees
- moved J8 11.8 mm to (54.5, 23.6)
- moved U5 7.45 mm to (30.0, 34.2)
- moved J4 2.00 mm to (31.9, 82.2)
- moved J5 2.00 mm to (39.7, 82.2)
- moved J3 2.00 mm to (24.0, 82.2)
- moved J6 2.00 mm to (47.6, 82.2)
- moved C11 0.42 mm to (34.8, 39.4)
Connections:
- C19 pad 1: GND -> VCC
- C19 pad 2: VCC -> GND
- SW1 pad 2: Net-(U1-EN) -> Net-(U1-IO0)
- U5 pad 1: unconnected-(U5-INT-Pad1) -> VCC
- U5 pad 10: GND -> VCC
- U5 pad 2: MAG_CS -> SPI_SCLK
- U5 pad 3: SPI_SCLK -> GND
- U5 pad 4: GND -> SPI_MOSI
- U5 pad 5: SPI_MOSI -> SPI_MISO
- U5 pad 6: SPI_MISO -> BARO_CS
Routing:
- net Net-(Q2-G): track 44.9 -> 80.4 mm, vias 2 -> 4
- net GND: track 379.4 -> 359.5 mm, vias 6 -> 5
- net SPI_SCLK: track 44.1 -> 25.8 mm, vias 4 -> 2
- net SPI_MISO: track 55.4 -> 47.7 mm
- net MAG_CS: track 6.69 -> 0.00 mm
- net +5V: track 104.0 -> 99.1 mm
- net SDA: track 40.0 -> 36.5 mm, vias 2 -> 1
- net BARO_CS: track 6.21 -> 2.83 mm
- net SPI_MOSI: track 42.2 -> 45.2 mm, vias 4 -> 3
- net GPIO2: track 29.2 -> 26.3 mm
- net SERVO1: track 75.9 -> 78.2 mm
- net SERVO3: track 52.5 -> 54.0 mm
- net SERVO4: track 55.5 -> 57.0 mm
- net SCL: track 31.2 -> 30.1 mm, vias 2 -> 1
- net NFVCC: track 106.7 -> 107.8 mm
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
Commit message: drc fixes
Parts:
- moved U7 0.61 mm to (37.1, 35.2)
- moved C6 0.20 mm to (27.4, 33.9)
Routing:
- net MAG_CS: track 0.00 -> 62.9 mm, vias 0 -> 4
- net IMU_CS: track 19.7 -> 79.9 mm, vias 2 -> 6
- net SERVO3: track 54.0 -> 96.8 mm, vias 0 -> 3
- net GND: track 359.5 -> 395.9 mm, vias 5 -> 9
- net SERVO1: track 78.2 -> 63.7 mm, vias 2 -> 1
- net Net-(Q2-G): track 80.4 -> 66.4 mm
- net SPI_MISO: track 47.7 -> 61.3 mm, vias 4 -> 5
- net SPI_SCLK: track 25.8 -> 36.1 mm, vias 2 -> 4
- net SERVO2: track 60.8 -> 67.5 mm
- net VCC: track 158.5 -> 161.0 mm, vias 4 -> 5
- net SPI_MOSI: track 45.2 -> 46.3 mm

Commit message: BOM + supply chain changes
Parts:
- removed SW3: TS-1088R-02026, easyeda2kicad:SW-SMD_L3.9-W3.0-P4.45
- added SW2: SW_Push, TL3365AF180QG:SW_TL3365AF180QG, F.Cu at (19.2, 23.8)
- P1: footprint Connector_USB:USB_C_Receptacle_HRO_TYPE-C-31-M-12 -> Connector_USB:USB_C_Receptacle_Amphenol_124019772112A
- SW1: value TS-1088R-02026 -> SW_Push; footprint easyeda2kicad:SW-SMD_L3.9-W3.0-P4.45 -> TL3365AF180QG:SW_TL3365AF180QG
- U7: footprint MLX90395KDC-BBA-001-SP:SOIC127P600X172-8N -> MLX90395KDC-BBA-101-SP:SOIC127P600X172-8N
- moved P1 1.07 mm to (17.4, 54.1)
- moved C6 0.41 mm to (27.5, 33.5)
- moved SW1 0.34 mm to (47.6, 34.9)
Routing:
- net +5V: track 99.1 -> 83.9 mm
- net IMU_CS: track 79.9 -> 74.7 mm
- net D+: track 29.7 -> 34.7 mm
- net SERVO2: track 67.5 -> 65.2 mm
- net GND: track 395.9 -> 397.9 mm
- net D-: track 31.8 -> 30.3 mm, vias 0 -> 2
- net Net-(P1-CC): track 3.03 -> 4.52 mm
- net Net-(U1-IO0): track 11.1 -> 10.1 mm

Commit message: fix conflict?
Parts:
- added L1: 3.3uh, Inductor_SMD:L_0805_2012Metric, F.Cu at (31.9, 63.0)
- R3: value 60 -> 10k
- R4: value 330 -> 54.9k
Connections:
- C18 pad 1: +5V -> Net-(U6-SW)
- U6 pad 2: +5V -> Net-(U6-SW)
Routing:
- net +5V: track 83.9 -> 87.8 mm
- net Net-(U6-SW): track 0.00 -> 3.49 mm
Changed lines of the file:
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@@
 	(net 58 "unconnected-(U7-A0-Pad5)")
 	(net 59 "unconnected-(U5-INT-Pad7)")
+	(net 60 "Net-(U6-SW)")
 	(footprint "TerminalBlock:TerminalBlock_Xinya_XY308-2.54-2P_1x02_P2.54mm_Horizontal"
 		(layer "F.Cu")
@@
 			)
 		)
-		(property "Value" "330"
+		(property "Value" "54.9k"
 			(at 0 1.43 90)
 			(layer "F.Fab")
@@
 			)
 		)
-		(property "Value" "60"
+		(property "Value" "10k"
 			(at 0 1.43 90)
 			(layer "F.Fab")
@@
 			(layers "F.Cu" "F.Mask" "F.Paste")
 			(roundrect_rratio 0.25)
-			(net 2 "+5V")
+			(net 60 "Net-(U6-SW)")
 			(pintype "passive")
 		)
@@
 		)
 	)
+	(footprint "Inductor_SMD:L_0805_2012Metric"
+		(layer "F.Cu")
+		(at 31.9375 63)
+		(descr "Inductor SMD 0805 (2012 Metric), square (rectangular) end terminal, IPC-7351 nominal, (Body size source: IPC-SM-782 page 80, https://www.pcb-3d.com/wordpress/wp-content/uploads/ipc-sm-782a_amendment_1_and_2.pdf), generated with kicad-footprint-generator")
+		(tags "inductor")
+		(property "Reference" "L1"
+			(at 0 -1.55 0)
+			(layer "F.SilkS")
+			(effects
+				(font
+					(size 1 1)
+					(thickness 0.15)
+				)
+			)
+		)
+		(property "Value" "3.3uh"
+			(at 0 1.55 0)
+			(layer "F.Fab")
+			(effects
+				(font
+					(size 1 1)
+					(thickness 0.15)
+				)
+			)
+		)
+		(property "Datasheet" "~"
+			(at 0 0 0)
+			(layer "F.Fab")
+			(hide yes)
+			(effects
+				(font
+					(size 1.27 1.27)
+					(thickness 0.15)
+				)
+			)
+		)
+		(property "Description" "Inductor"
+			(at 0 0 0)
+			(layer "F.Fab")
+			(hide yes)
+			(effects
+				(font
+					(size 1.27 1.27)
+					(thickness 0.15)
+				)
+			)
+		)
+		(property ki_fp_filters "Choke_* *Coil* Inductor_* L_*")
+		(sheetname "/")
+		(sheetfile "Sigma1.kicad_sch")
+		(attr smd)
+		(fp_line
+			(start -0.399622 -0.56)
+			(end 0.399622 -0.56)
+			(stroke
+				(width 0.12)
+				(type solid)
+			)
+			(layer "F.SilkS")
+		)
+		(fp_line
+			(start -0.399622 0.56)
+			(end 0.399622 0.56)
+			(stroke
+				(width 0.12)
+				(type solid)
+			)
+			(layer "F.SilkS")
+		)
+		(fp_line
+			(start -1.75 -0.85)
+			(end 1.75 -0.85)
+			(stroke
+				(width 0.05)
+				(type solid)
+			)
+			(layer "F.CrtYd")
+		)
+		(fp_line
+			(start -1.75 0.85)
+			(end -1.75 -0.85)
+			(stroke
+				(width 0.05)
+				(type solid)
+			)
+			(layer "F.CrtYd")
+		)
+		(fp_line
+			(start 1.75 -0.85)
+			(end 1.75 0.85)
+			(stroke
+				(width 0.05)
+				(type solid)
+			)
+			(layer "F.CrtYd")
+		)
+		(fp_line
+			(start 1.75 0.85)
+			(end -1.75 0.85)
+			(stroke
+				(width 0.05)
+				(type solid)
+			)
+			(layer "F.CrtYd")
+		)
+		(fp_line
+			(start -1 -0.45)
+			(end 1 -0.45)
+			(stroke
+				(width 0.1)
+				(type solid)
+			)
+			(layer "F.Fab")
+		)
+		(fp_line
+			(start -1 0.45)
+			(end -1 -0.45)
+			(stroke
+				(width 0.1)
+				(type solid)
+			)
+			(layer "F.Fab")
+		)
+		(fp_line
+			(start 1 -0.45)
+			(end 1 0.45)
+			(stroke
+				(width 0.1)
+				(type solid)
+			)
+			(layer "F.Fab")
+		)
+		(fp_line
+			(start 1 0.45)
+			(end -1 0.45)
+			(stroke
+				(width 0.1)
+				(type solid)
+			)
+			(layer "F.Fab")
+		)
+		(fp_text user "${REFERENCE}"
+			(at 0 0 0)
+			(layer "F.Fab")
+			(effects
+				(font
+					(size 0.5 0.5)
+					(thickness 0.08)
+				)
+			)
+		)
+		(pad "1" smd roundrect
+			(at -1.0625 0)
+			(size 0.875 1.2)
+			(layers "F.Cu" "F.Mask" "F.Paste")
+			(roundrect_rratio 0.25)
+			(net 2 "+5V")
+			(pinfunction "1")
+			(pintype "passive")
+		)
+		(pad "2" smd roundrect
+			(at 1.0625 0)
+			(size 0.875 1.2)
+			(layers "F.Cu" "F.Mask" "F.Paste")
+			(roundrect_rratio 0.25)
+			(net 60 "Net-(U6-SW)")
+			(pinfunction "2")
+			(pintype "passive")
+		)
+		(embedded_fonts no)
+		(model "${KICAD9_3DMODEL_DIR}/Inductor_SMD.3dshapes/L_0805_2012Metric.step"
+			(offset
+				(xyz 0 0 0)
+			)
+			(scale
+				(xyz 1 1 1)
+			)
+			(rotate
+				(xyz 0 0 0)
+			)
+		)
+	)
 	(footprint "Capacitor_SMD:C_0603_1608Metric"
 		(layer "F.Cu")
@@
 			(layers "F.Cu" "F.Mask" "F.Paste")
 			(roundrect_rratio 0.25)
-			(net 2 "+5V")
+			(net 60 "Net-(U6-SW)")
 			(pinfunction "SW")
 			(pintype "output")
@@
 	)
 	(segment
+		(start 27.034 66.449)
+		(end 30 66.449)
+		(width 0.2)
+		(layer "F.Cu")
+		(net 2)
+	)
+	(segment
 		(start 25.275 62.025)
 		(end 25.3 62)
@@
 	)
 	(segment
-		(start 27.034 66.449)
+		(start 30 66.449)
 		(end 31.974 66.449)
 		(width 0.2)
@@
 	)
 	(segment
+		(start 30.875 63)
+		(end 30.875 65.574)
+		(width 0.2)
+		(layer "F.Cu")
+		(net 2)
+	)
+	(segment
 		(start 25.27 84.76)
 		(end 23.99 84.76)
@@
 	)
 	(segment
+		(start 30.875 65.574)
+		(end 30 66.449)
+		(width 0.2)
+		(layer "F.Cu")
+		(net 2)
+	)
+	(segment
 		(start 31.9 71.8125)
 		(end 31.9 77.4283)
@@
 		(net 49)
 	)
+	(segment
+		(start 33 65.475)
+		(end 32.28355 66.19145)
+		(width 0.2)
+		(layer "F.Cu")
+		(net 60)
+	)
+	(segment
+		(start 33 63)
+		(end 33 65.475)
+		(width 0.2)
+		(layer "F.Cu")
+		(net 60)
+	)
 	(embedded_fonts no)
